File: kicad/main.kicad_sch (KiCad schematic)
At the start: 118 parts, among them IC1 H616, IC2 AR1100_SSOP, IC3 KLMAG1JETD-B041, IC4 RTL8723DS-CG, IC5 TFP401PZP, J1 AudioJack4, J11 USB_A, J12 USB_A, J2 USB_C_Receptacle_USB2.0_16P, J3 USB_C_Receptacle_USB2.0_16P, J4 Conn_01x40_Pin, J9 HDMI_D_1.4, Q1 BSS138, U1 K4UBE3D4AB-MGCL, U2 1.1v, U3 1.8v, U4 0.6v, U5 24LC02BT-I/OT, U6 LT1117(3V3), U7 TFP401, U8 FAN5333BSX, X1 47151-0001, X2 microUSB, X3 XF2-40-RARBT, Y1 12MHz

Commit message: traces
Parts:
- added C29: C1uf, symbol Device:C
- added U9: buck boost converters 3.3v, Converter_DCDC:Converter_DCDC_TRACO_TSR0.6-48xxWI_TSR0.6-48xxxWI_THT, symbol Converter_DCDC:TSR0.6-4833WI
- added decupple: 1.8v, Converter_DCDC:Converter_DCDC_TRACO_TSR0.6-48xxWI_TSR0.6-48xxxWI_THT, symbol Converter_DCDC:TSR0.6-4833WI
Connections:
- net 1.8v dram: now also decupple.1 (Vin); no longer U3.3 (Vout)
- net GND: now also IC3.H10 (VSS_5), C29.1
- net at BT1.1 (+), U2.1 (Vin), U3.1 (Vin)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: now also U9.3 (Vout)
- net at IC3.C2 (VDDI): now also C29.2
- net 3.3v: now reaches IC3.J10 (VDDF_3)
- net 1.8v: now reaches IC3.M4 (VDD_2)
- net PH: now reaches IC1.A12 (PH9)
- net PH: now also IC1.A14 (PH4), IC1.B12 (PH7), IC1.B13 (PH10), IC1.B14 (PH5), IC1.B15 (PH2), IC1.C13 (PH8), IC1.C14 (PH6), IC1.C15 (PH3), IC1.D15 (PH1), IC1.D16 (PH0)
- net PI: now reaches IC1.D4 (PI1)
- net PI: now also IC1.D5 (PI9), IC1.E4 (PI3), IC1.E5 (PI13), IC1.E6 (PI8), IC1.G4 (PI7), IC1.G5 (PI4), IC1.G6 (PI2), IC1.H4 (PI5), IC1.H5 (PI6), IC1.H6 (PI0), IC1.J6 (VCC_PI), IC1.K4 (PI11), IC1.K5 (PI12), IC1.K6 (PI16), IC1.L2 (PF4), IC1.L3 (PF5), IC1.L4 (PI15), IC1.L5 (PI10), IC1.L6 (PI14)
- net PF: now reaches IC1.J2 (PF0)
- net PF: now also IC1.J3 (PF1), IC1.K1 (PF2), IC1.K2 (PF6), IC1.K3 (PF3)
- new net: U3.3 (Vout), decupple.2 (GND)
- new net 1.8v EMMC: decupple.3 (Vout)
- new net 3.3v EMMC VDDF: U9.1 (Vin)
